File: fst-01.sch (KiCad schematic (older format))
At the start: 22 parts, among them J1 USB_A, K1 CONN_3, K2 CONN_3, U1 STM32F103CB, U2 CAT6217-330, U3 STF202-22, X1 8MHz

Commit message: fix STF-202 connection
Connections:
- wire segments 92 -> 94
Changed lines of the file:
@@
-EESchema Schematic File Version 2  date Tue 09 Aug 2011 18:16:34 JST
+EESchema Schematic File Version 2  date Wed 17 Aug 2011 13:39:00 JST
 LIBS:device
 LIBS:stm32f103
@@
 Sheet 1 1
 Title ""
-Date "9 aug 2011"
+Date "17 aug 2011"
 Rev ""
 Comp ""
@@
 Comment4 ""
 $EndDescr
-Wire Wire Line
-	7525 5600 6850 5600
-Wire Wire Line
-	6850 5600 6850 4850
-Wire Wire Line
-	6850 4850 6450 4850
+Connection ~ 7750 3650
+Wire Wire Line
+	7750 4300 7750 3350
+Wire Wire Line
+	3950 4150 3950 3900
+Wire Wire Line
+	4125 6375 4125 6525
+Wire Wire Line
+	5750 2800 5750 3450
+Wire Wire Line
+	7650 3350 7650 3500
+Connection ~ 7750 3350
+Wire Wire Line
+	7050 2150 7050 2250
+Wire Wire Line
+	5850 3025 5850 2800
+Wire Wire Line
+	4125 6525 4450 6525
+Wire Wire Line
+	4450 6525 4450 6575
+Wire Wire Line
+	6450 4350 7250 4350
+Wire Wire Line
+	7250 4350 7250 3400
+Wire Wire Line
+	7250 3400 5950 3400
+Wire Wire Line
+	9650 4850 9450 4850
+Wire Wire Line
+	9650 5150 9500 5150
+Wire Wire Line
+	9500 5150 9500 5300
+Wire Wire Line
+	7750 4300 8550 4300
+Wire Wire Line
+	4450 6275 4450 6375
+Wire Wire Line
+	4450 6375 4225 6375
+Wire Wire Line
+	8025 5600 8100 5600
+Wire Wire Line
+	5200 3225 5200 3175
+Wire Wire Line
+	5200 3175 5050 3175
+Wire Wire Line
+	5350 5950 5350 6100
+Wire Wire Line
+	6450 4150 6450 3900
+Connection ~ 3200 5400
+Wire Wire Line
+	3200 5400 3200 4750
+Wire Wire Line
+	3200 4750 3950 4750
+Wire Wire Line
+	2700 5400 2700 5300
+Wire Wire Line
+	3950 4550 3100 4550
+Connection ~ 6400 5950
+Wire Wire Line
+	6600 5950 6400 5950
+Wire Wire Line
+	3800 4950 3800 5250
+Wire Wire Line
+	3800 4950 3950 4950
+Wire Wire Line
+	5650 5950 5650 6150
+Wire Wire Line
+	6600 5950 6600 6050
+Wire Wire Line
+	6400 5950 6400 6150
+Connection ~ 4550 3050
+Wire Wire Line
+	4315 3050 4750 3050
+Wire Wire Line
+	4315 3050 4315 3140
+Wire Wire Line
+	4750 3050 4750 3450
+Connection ~ 4550 3450
+Wire Wire Line
+	3550 4150 3450 4150
+Wire Wire Line
+	3450 4150 3450 4250
+Wire Wire Line
+	7200 2700 7200 2650
+Wire Wire Line
+	7950 3750 7950 3800
+Wire Wire Line
+	8150 2250 8150 2400
+Connection ~ 7200 2250
+Wire Wire Line
+	2450 4300 2375 4300
+Wire Wire Line
+	2375 4300 2375 4450
+Connection ~ 2850 4300
+Wire Wire Line
+	2850 4300 3100 4300
+Wire Wire Line
+	3100 4300 3100 4550
+Wire Wire Line
+	7950 4950 7550 4950
+Wire Wire Line
+	7550 4950 7550 4550
+Wire Wire Line
+	7550 4550 6450 4550
+Wire Wire Line
+	9650 4950 8950 4950
+Wire Wire Line
+	8950 4850 8950 4650
+Wire Wire Line
+	9050 4300 9450 4300
+Wire Wire Line
+	8850 4700 8850 4650
+Wire Wire Line
+	8850 4650 8950 4650
+Wire Wire Line
+	8950 5050 9650 5050
+Wire Wire Line
+	6450 4450 7450 4450
+Wire Wire Line
+	7450 4450 7450 5050
+Wire Wire Line
+	7450 5050 7950 5050
+Wire Wire Line
+	3100 4900 3100 4650
+Wire Wire Line
+	3100 4900 2850 4900
+Connection ~ 2850 4900
+Wire Wire Line
+	2375 5050 2375 4900
+Wire Wire Line
+	2375 4900 2450 4900
+Connection ~ 6450 4050
+Wire Wire Line
+	6450 4250 6850 4250
+Wire Wire Line
+	6850 4250 6850 4050
+Wire Wire Line
+	7050 4150 7050 4050
+Wire Wire Line
+	7050 4050 6850 4050
+Connection ~ 6850 4050
+Wire Wire Line
+	4225 3385 4225 3450
+Wire Wire Line
+	4225 3450 4650 3450
+Connection ~ 3950 4150
+Wire Wire Line
+	3700 4950 3700 4850
+Wire Wire Line
+	3950 4850 3500 4850
+Connection ~ 3700 4850
+Wire Wire Line
+	3800 5250 3300 5250
+Wire Wire Line
+	3300 5250 3300 5200
+Connection ~ 3500 5250
+Wire Wire Line
+	6000 5950 5750 5950
+Wire Wire Line
+	6400 6150 5650 6150
+Wire Wire Line
+	6450 4050 6450 4050
+Wire Wire Line
+	3100 4650 3950 4650
+Wire Wire Line
+	3200 5800 3200 5900
+Wire Wire Line
+	5050 3175 5050 3450
+Wire Wire Line
+	8100 6000 8100 6100
+Wire Wire Line
+	9450 4300 9450 4850
+Wire Wire Line
+	4025 6375 4025 6675
+Wire Wire Line
+	4025 6675 5150 6675
+Wire Wire Line
+	5150 6675 5150 5950
+Wire Wire Line
+	7750 3350 7950 3350
+Wire Wire Line
+	7550 3350 7550 3650
+Wire Wire Line
+	7550 3650 7750 3650
+Wire Wire Line
+	7050 2250 7550 2250
+Wire Wire Line
+	5950 3400 5950 2800
+Wire Wire Line
+	5950 5850 5950 5950
 Connection ~ 5950 5950
 Wire Wire Line
-	5950 5850 5950 5950
-Wire Wire Line
-	5950 2800 5950 3400
-Connection ~ 7750 4300
-Wire Wire Line
-	7550 2250 7050 2250
-Connection ~ 7750 3650
-Wire Wire Line
-	7750 3650 7550 3650
-Wire Wire Line
-	7550 3650 7550 3350
-Wire Wire Line
-	7950 3350 7750 3350
-Wire Wire Line
-	5150 5950 5150 6675
-Wire Wire Line
-	5150 6675 4025 6675
-Wire Wire Line
-	4025 6675 4025 6375
-Wire Wire Line
-	9450 4300 9450 4850
-Wire Wire Line
-	8100 6000 8100 6100
-Wire Wire Line
-	5050 3450 5050 3175
-Wire Wire Line
-	3200 5800 3200 5900
-Wire Wire Line
-	3950 4650 3100 4650
-Wire Wire Line
-	6450 4050 6450 4050
-Wire Wire Line
-	6400 6150 5650 6150
-Wire Wire Line
-	6000 5950 5750 5950
-Connection ~ 3500 5250
-Wire Wire Line
-	3300 5200 3300 5250
-Wire Wire Line
-	3300 5250 3800 5250
-Connection ~ 3700 4850
-Wire Wire Line
-	3950 4850 3500 4850
-Wire Wire Line
-	3700 4950 3700 4850
-Connection ~ 3950 4150
-Wire Wire Line
-	4650 3450 4225 3450
-Wire Wire Line
-	4225 3450 4225 3385
-Connection ~ 6850 4050
-Wire Wire Line
-	7050 4050 6850 4050
-Wire Wire Line
-	7050 4050 7050 4150
-Wire Wire Line
-	6850 4050 6850 4250
-Wire Wire Line
-	6850 4250 6450 4250
-Connection ~ 6450 4050
-Wire Wire Line
-	2450 4900 2375 4900
-Wire Wire Line
-	2375 4900 2375 5050
-Connection ~ 2850 4900
-Wire Wire Line
-	2850 4900 3100 4900
-Wire Wire Line
-	3100 4900 3100 4650
-Wire Wire Line
-	7950 5050 7450 5050
-Wire Wire Line
-	7450 5050 7450 4450
-Wire Wire Line
-	7450 4450 6450 4450
-Wire Wire Line
-	8950 5050 9650 5050
-Wire Wire Line
-	8850 4650 8950 4650
-Wire Wire Line
-	8850 4650 8850 4700
-Wire Wire Line
-	9450 4300 9050 4300
-Wire Wire Line
-	8950 4650 8950 4850
-Wire Wire Line
-	9650 4950 8950 4950
-Wire Wire Line
-	6450 4550 7550 4550
-Wire Wire Line
-	7550 4550 7550 4950
-Wire Wire Line
-	7550 4950 7950 4950
-Wire Wire Line
-	3100 4300 3100 4550
-Wire Wire Line
-	3100 4300 2850 4300
-Connection ~ 2850 4300
-Wire Wire Line
-	2375 4450 2375 4300
-Wire Wire Line
-	2375 4300 2450 4300
-Connection ~ 7200 2250
-Wire Wire Line
-	8150 2250 8150 2400
-Wire Wire Line
-	7950 3750 7950 3800
-Wire Wire Line
-	7200 2700 7200 2650
-Wire Wire Line
-	3450 4250 3450 4150
-Wire Wire Line
-	3450 4150 3550 4150
-Connection ~ 4550 3450
-Wire Wire Line
-	4750 3450 4750 3050
-Wire Wire Line
-	4315 3140 4315 3050
-Wire Wire Line
-	4315 3050 4750 3050
-Connection ~ 4550 3050
-Wire Wire Line
-	6400 6150 6400 5950
-Wire Wire Line
-	6600 6050 6600 5950
-Wire Wire Line
-	5650 6150 5650 5950
-Wire Wire Line
-	3950 4950 3800 4950
-Wire Wire Line
-	3800 4950 3800 5250
-Wire Wire Line
-	6600 5950 6400 5950
-Connection ~ 6400 5950
-Wire Wire Line
-	3100 4550 3950 4550
-Wire Wire Line
-	2700 5400 2700 5300
-Wire Wire Line
-	3950 4750 3200 4750
-Wire Wire Line
-	3200 4750 3200 5400
-Connection ~ 3200 5400
-Wire Wire Line
-	6450 4150 6450 3900
-Wire Wire Line
-	5350 5950 5350 6100
-Wire Wire Line
-	5050 3175 5200 3175
-Wire Wire Line
-	5200 3175 5200 3225
-Wire Wire Line
-	8025 5600 8100 5600
-Wire Wire Line
-	4225 6375 4450 6375
-Wire Wire Line
-	4450 6375 4450 6275
-Wire Wire Line
-	7750 4300 8550 4300
-Wire Wire Line
-	9500 5300 9500 5150
-Wire Wire Line
-	9500 5150 9650 5150
-Wire Wire Line
-	9450 4850 9650 4850
-Wire Wire Line
-	5950 3400 7250 3400
-Wire Wire Line
-	7250 3400 7250 4350
-Wire Wire Line
-	7250 4350 6450 4350
-Wire Wire Line
-	4450 6575 4450 6525
-Wire Wire Line
-	4450 6525 4125 6525
-Wire Wire Line
-	5850 3025 5850 2800
-Wire Wire Line
-	7950 4850 7750 4850
-Wire Wire Line
-	7750 4850 7750 3350
-Wire Wire Line
-	7050 2250 7050 2150
-Connection ~ 7750 3350
-Wire Wire Line
-	7650 3350 7650 3500
-Wire Wire Line
-	5750 2800 5750 3450
-Wire Wire Line
-	4125 6525 4125 6375
-Wire Wire Line
-	3950 4150 3950 3900
+	6450 4850 6850 4850
+Wire Wire Line
+	6850 4850 6850 5600
+Wire Wire Line
+	6850 5600 7525 5600
+Wire Wire Line
+	6450 4650 7650 4650
+Wire Wire Line
+	7650 4650 7650 4850
+Wire Wire Line
+	7650 4850 7950 4850
 Text Label 7500 5600 2    60   ~ 0
 LED

Commit message: Use NUF2221 instead of STF202
Parts:
- removed U3: STF202-22, symbol STF202-22
- added U3: NUF2221W1, symbol NUF2221W1
Connections:
- wire segments 94 -> 98

Commit message: Fix NUF2221 connection
Connections:
- wire segments 98 -> 96
Changed lines of the file:
@@
-EESchema Schematic File Version 2  date Mon 22 Aug 2011 17:45:11 JST
+EESchema Schematic File Version 2  date Mon 05 Sep 2011 12:27:27 JST
 LIBS:device
 LIBS:stm32f103
@@
 Sheet 1 1
 Title ""
-Date "22 aug 2011"
+Date "5 sep 2011"
 Rev ""
 Comp ""
@@
 $EndDescr
 Wire Wire Line
-	9650 5050 9200 5050
-Wire Wire Line
-	9100 5000 9100 4950
-Wire Wire Line
-	8950 4850 9400 4850
-Wire Wire Line
-	7950 4850 7550 4850
-Wire Wire Line
-	7550 4850 7550 4550
-Wire Wire Line
-	6450 4650 7650 4650
-Wire Wire Line
-	7525 5600 6850 5600
-Wire Wire Line
-	6850 5600 6850 4850
-Wire Wire Line
-	6850 4850 6450 4850
+	8950 4950 9200 4950
+Wire Wire Line
+	9200 4950 9200 4650
+Wire Wire Line
+	9200 4650 6450 4650
+Wire Wire Line
+	8950 5050 9650 5050
+Wire Wire Line
+	7950 5050 7950 5300
+Wire Wire Line
+	7950 5300 7650 5300
+Wire Wire Line
+	9650 4950 9400 4950
+Wire Wire Line
+	9400 4950 9400 4850
+Connection ~ 7750 3650
+Wire Wire Line
+	7750 4300 7750 3350
+Wire Wire Line
+	3950 4150 3950 3900
+Wire Wire Line
+	4125 6375 4125 6525
+Wire Wire Line
+	5750 2800 5750 3450
+Wire Wire Line
+	7650 3350 7650 3500
+Connection ~ 7750 3350
+Wire Wire Line
+	7050 2150 7050 2250
+Wire Wire Line
+	5850 3025 5850 2800
+Wire Wire Line
+	4125 6525 4450 6525
+Wire Wire Line
+	4450 6525 4450 6575
+Wire Wire Line
+	6450 4350 7250 4350
+Wire Wire Line
+	7250 4350 7250 3400
+Wire Wire Line
+	7250 3400 5950 3400
+Wire Wire Line
+	9650 4850 9450 4850
+Wire Wire Line
+	9650 5150 9500 5150
+Wire Wire Line
+	9500 5150 9500 5300
+Wire Wire Line
+	7750 4300 8550 4300
+Wire Wire Line
+	4450 6275 4450 6375
+Wire Wire Line
+	4450 6375 4225 6375
+Wire Wire Line
+	8025 5600 8100 5600
+Wire Wire Line
+	5200 3225 5200 3175
+Wire Wire Line
+	5200 3175 5050 3175
+Wire Wire Line
+	5350 5950 5350 6100
+Wire Wire Line
+	6450 4150 6450 3900
+Connection ~ 3200 5400
+Wire Wire Line
+	3200 5400 3200 4750
+Wire Wire Line
+	3200 4750 3950 4750
+Wire Wire Line
+	2700 5400 2700 5300
+Wire Wire Line
+	3950 4550 3100 4550
+Connection ~ 6400 5950
+Wire Wire Line
+	6600 5950 6400 5950
+Wire Wire Line
+	3800 4950 3800 5250
+Wire Wire Line
+	3800 4950 3950 4950
+Wire Wire Line
+	5650 5950 5650 6150
+Wire Wire Line
+	6600 5950 6600 6050
+Wire Wire Line
+	6400 5950 6400 6150
+Connection ~ 4550 3050
+Wire Wire Line
+	4315 3050 4750 3050
+Wire Wire Line
+	4315 3050 4315 3140
+Wire Wire Line
+	4750 3050 4750 3450
+Connection ~ 4550 3450
+Wire Wire Line
+	3550 4150 3450 4150
+Wire Wire Line
+	3450 4150 3450 4250
+Wire Wire Line
+	7200 2700 7200 2650
+Wire Wire Line
+	7950 3750 7950 3800
+Wire Wire Line
+	8150 2250 8150 2400
+Connection ~ 7200 2250
+Wire Wire Line
+	2450 4300 2375 4300
+Wire Wire Line
+	2375 4300 2375 4450
+Connection ~ 2850 4300
+Wire Wire Line
+	2850 4300 3100 4300
+Wire Wire Line
+	3100 4300 3100 4550
+Wire Wire Line
+	6450 4550 7550 4550
+Wire Wire Line
+	9050 4300 9450 4300
+Wire Wire Line
+	3100 4900 3100 4650
+Wire Wire Line
+	3100 4900 2850 4900
+Connection ~ 2850 4900
+Wire Wire Line
+	2375 5050 2375 4900
+Wire Wire Line
+	2375 4900 2450 4900
+Connection ~ 6450 4050
+Wire Wire Line
+	6450 4250 6850 4250
+Wire Wire Line
+	6850 4250 6850 4050
+Wire Wire Line
+	7050 4150 7050 4050
+Wire Wire Line
+	7050 4050 6850 4050
+Connection ~ 6850 4050
+Wire Wire Line
+	4225 3385 4225 3450
+Wire Wire Line
+	4225 3450 4650 3450
+Connection ~ 3950 4150
+Wire Wire Line
+	3700 4950 3700 4850
+Wire Wire Line
+	3950 4850 3500 4850
+Connection ~ 3700 4850
+Wire Wire Line
+	3800 5250 3300 5250
+Wire Wire Line
+	3300 5250 3300 5200
+Connection ~ 3500 5250
+Wire Wire Line
+	6000 5950 5750 5950
+Wire Wire Line
+	6400 6150 5650 6150
+Wire Wire Line
+	6450 4050 6450 4050
+Wire Wire Line
+	3100 4650 3950 4650
+Wire Wire Line
+	3200 5800 3200 5900
+Wire Wire Line
+	5050 3175 5050 3450
+Wire Wire Line
+	8100 6000 8100 6100
+Wire Wire Line
+	9450 4300 9450 4850
+Wire Wire Line
+	4025 6375 4025 6675
+Wire Wire Line
+	4025 6675 5150 6675
+Wire Wire Line
+	5150 6675 5150 5950
+Wire Wire Line
+	7750 3350 7950 3350
+Wire Wire Line
+	7550 3350 7550 3650
+Wire Wire Line
+	7550 3650 7750 3650
+Wire Wire Line
+	7050 2250 7550 2250
+Wire Wire Line
+	5950 3400 5950 2800
+Wire Wire Line
+	5950 5850 5950 5950
 Connection ~ 5950 5950
 Wire Wire Line
-	5950 5850 5950 5950
-Wire Wire Line
-	5950 2800 5950 3400
-Wire Wire Line
-	7550 2250 7050 2250
-Wire Wire Line
-	7750 3650 7550 3650
-Wire Wire Line
-	7550 3650 7550 3350
-Wire Wire Line
-	7950 3350 7750 3350
-Wire Wire Line
-	5150 5950 5150 6675
-Wire Wire Line
-	5150 6675 4025 6675
-Wire Wire Line
-	4025 6675 4025 6375
-Wire Wire Line
-	9450 4300 9450 4850
-Wire Wire Line
-	8100 6000 8100 6100
-Wire Wire Line
-	5050 3450 5050 3175
-Wire Wire Line
-	3200 5800 3200 5900
-Wire Wire Line
-	3950 4650 3100 4650
-Wire Wire Line
-	6450 4050 6450 4050
-Wire Wire Line
-	6400 6150 5650 6150
-Wire Wire Line
-	5750 5950 6000 5950
-Connection ~ 3500 5250
-Wire Wire Line
-	3300 5200 3300 5250
-Wire Wire Line
-	3300 5250 3800 5250
-Connection ~ 3700 4850
-Wire Wire Line
-	3500 4850 3950 4850
-Wire Wire Line
-	3700 4950 3700 4850
-Connection ~ 3950 4150
-Wire Wire Line
-	4650 3450 4225 3450
-Wire Wire Line
-	4225 3450 4225 3385
-Connection ~ 6850 4050
-Wire Wire Line
-	7050 4050 6850 4050
-Wire Wire Line
-	7050 4050 7050 4150
-Wire Wire Line
-	6850 4050 6850 4250
-Wire Wire Line
-	6850 4250 6450 4250
-Connection ~ 6450 4050
-Wire Wire Line
-	2450 4900 2375 4900
-Wire Wire Line
-	2375 4900 2375 5050
-Connection ~ 2850 4900
-Wire Wire Line
-	2850 4900 3100 4900
-Wire Wire Line
-	3100 4900 3100 4650
-Wire Wire Line
-	7950 5050 7450 5050
-Wire Wire Line
-	7450 5050 7450 4450
-Wire Wire Line
-	7450 4450 6450 4450
-Wire Wire Line
-	9100 4950 8950 4950
-Wire Wire Line
-	9450 4300 9050 4300
-Wire Wire Line
-	7550 4550 6450 4550
-Wire Wire Line
-	3100 4300 3100 4550
-Wire Wire Line
-	3100 4300 2850 4300
-Connection ~ 2850 4300
-Wire Wire Line
-	2375 4450 2375 4300
-Wire Wire Line
-	2375 4300 2450 4300
-Connection ~ 7200 2250
-Wire Wire Line
-	8150 2250 8150 2400
-Wire Wire Line
-	7950 3750 7950 3800
-Wire Wire Line
-	7200 2700 7200 2650
-Wire Wire Line
-	3450 4250 3450 4150
-Wire Wire Line
-	3450 4150 3550 4150
-Connection ~ 4550 3450
-Wire Wire Line
-	4750 3450 4750 3050
-Wire Wire Line
-	4315 3140 4315 3050
-Wire Wire Line
-	4315 3050 4750 3050
-Connection ~ 4550 3050
-Wire Wire Line
-	6400 6150 6400 5950
-Wire Wire Line
-	6600 6050 6600 5950
-Wire Wire Line
-	5650 6150 5650 5950
-Wire Wire Line
-	3950 4950 3800 4950
-Wire Wire Line
-	3800 4950 3800 5250
-Wire Wire Line
-	6600 5950 6400 5950
-Connection ~ 6400 5950
-Wire Wire Line
-	3100 4550 3950 4550
-Wire Wire Line
-	2700 5400 2700 5300
-Wire Wire Line
-	3950 4750 3200 4750
-Wire Wire Line
-	3200 4750 3200 5400
-Connection ~ 3200 5400
-Wire Wire Line
-	6450 3900 6450 4150
-Wire Wire Line
-	5350 5950 5350 6100
-Wire Wire Line
-	5050 3175 5200 3175
-Wire Wire Line
-	5200 3175 5200 3225
-Wire Wire Line
-	8025 5600 8100 5600
-Wire Wire Line
-	4225 6375 4450 6375
-Wire Wire Line
-	4450 6375 4450 6275
-Wire Wire Line
-	8550 4300 7750 4300
-Wire Wire Line
-	9500 5300 9500 5150
-Wire Wire Line
-	9500 5150 9650 5150
-Wire Wire Line
-	9450 4850 9650 4850
-Wire Wire Line
-	5950 3400 7250 3400
-Wire Wire Line
-	7250 3400 7250 4350
-Wire Wire Line
-	7250 4350 6450 4350
-Wire Wire Line
-	4450 6575 4450 6525
-Wire Wire Line
-	4450 6525 4125 6525
-Wire Wire Line
-	5850 3025 5850 2800
-Wire Wire Line
-	7050 2250 7050 2150
-Connection ~ 7750 3350
-Wire Wire Line
-	7650 3350 7650 3500
-Wire Wire Line
-	5750 2800 5750 3450
-Wire Wire Line
-	4125 6525 4125 6375
-Wire Wire Line
-	3950 4150 3950 3900
-Wire Wire Line
-	7750 4300 7750 3350
-Connection ~ 7750 3650
-Wire Wire Line
-	7650 4650 7650 4950
-Wire Wire Line
-	7650 4950 7950 4950
-Wire Wire Line
-	9400 4850 9400 4950
-Wire Wire Line
-	9400 4950 9650 4950
-Wire Wire Line
-	8950 5050 8950 5200
-Wire Wire Line
-	8950 5200 9200 5200
-Wire Wire Line
-	9200 5200 9200 5050
+	6450 4850 6850 4850
+Wire Wire Line
+	6850 4850 6850 5600
+Wire Wire Line
+	6850 5600 7525 5600
+Wire Wire Line
+	7550 4550 7550 4850
+Wire Wire Line
+	7550 4850 7950 4850
+Wire Wire Line
+	9400 4850 8950 4850
+Wire Wire Line
+	7950 4950 7850 4950
+Wire Wire Line
+	7850 4950 7850 5000
+Wire Wire Line
+	6450 4450 7650 4450
+Wire Wire Line
+	7650 4450 7650 5300
 $Comp
 L NUF2221W1 U3
@@
 F 1 "NUF2221W1" H 8450 4725 70  0000 C CNN
 	1    8450 4950
-	-1   0    0    1
+	1    0    0    1
 $EndComp
 Text Label 7500 5600 2    60   ~ 0
 LED
-Text Label 7700 5050 2    60   ~ 0
+Text Label 7650 5050 2    60   ~ 0
 D+
 Text Label 7850 4850 2    60   ~ 0
@@
 L GND #PWR026
 U 1 1 4E2CCCBB
-P 9100 5000
-F 0 "#PWR026" H 9100 5000 30  0001 C CNN
-F 1 "GND" H 9100 4930 30  0001 C CNN
-	1    9100 5000
-	1    0    0    -1
-$EndComp
+P 7850 5000
+F 0 "#PWR026" H 7850 5000 30  0001 C CNN
+F 1 "GND" H 7850 4930 30  0001 C CNN
+	1    7850 5000
+	1    0    0    -1
+$EndComp

Commit message: Major change: QFN36
Parts:
- removed C6: 0.1uF, symbol C
- removed F1: RESETTABLE FUSE, symbol FUSE
- removed K1: CONN_3, symbol CONN_3
- removed R1: 100k, symbol R
- removed U1: STM32F103CB, symbol STM32F103CB
- added K1: CONN_4, symbol CONN_4
- added K3: CONN_3, symbol CONN_3
- added U1: STM32F103TB, symbol STM32F103TB
- C10: value 1uF -> 4.7uF
- C8: renamed from C9; value 1uF -> 4.7uF
- renumbered C7 to C6, C8 to C7, C11 to C9, R2 to R1
Connections:
- net labels added: PA2, PA3, PA5, PA6, PA7, USB_EN
- net labels removed: PB0, VBUS_PLUG
- wire segments 96 -> 100
Other:
- moved on the sheet: C1, C2, C3, C4, C5, C6

Commit message: Change for SPI flash memory and small XTAL
Parts:
- removed K1: CONN_4, symbol CONN_4
- removed K3: CONN_3, symbol CONN_3
- added C11: 0.1uF, symbol C
- added K2, K3: CONN_2, symbol CONN_2
- added U4: SST25VF032B, symbol SST25VF032B
- X1: value 8MHz -> 12MHz
- renumbered K2 to K1
Connections:
- net labels added: CLK, MISO, MOSI, NSS
- net labels removed: PA5, PA6, PA7
- wire segments 100 -> 108
Other:
- moved on the sheet: D1, R1

Commit message: change +3V3 part in schematic.
Connections:
- net labels added: +3V3
- net labels removed: +3,3V

Commit message: change parts of connectors
Parts:
- J1: symbol USB_2 -> USB_A
- K1: symbol CONN_3 -> CONN_01X03
- K2, K3: symbol CONN_2 -> CONN_01X02
Changed lines of the file:
@@
 LIBS:conn
 LIBS:sst25vf032b
+LIBS:fst-01-cache
 EELAYER 25 0
 EELAYER END
@@
 $EndDescr
 $Comp
-L CONN_2 K3
+L CONN_01X02 K3
 U 1 1 4E8424A4
 P 3125 6200
@@
 $EndComp
 $Comp
-L CONN_2 K2
+L CONN_01X02 K2
 U 1 1 4E84249C
 P 2450 5725
@@
 GND
 $Comp
-L CONN_3 K1
+L CONN_01X03 K1
 U 1 1 4E32185E
-P 5850 2450
-F 0 "K1" V 5800 2450 50  0000 C CNN
-F 1 "CONN_3" V 5900 2450 40  0000 C CNN
-F 2 "" H 5850 2450 60  0001 C CNN
-F 3 "" H 5850 2450 60  0001 C CNN
-	1    5850 2450
+P 5850 2600
+F 0 "K1" V 5800 2600 50  0000 C CNN
+F 1 "CONN_3" V 5900 2600 40  0000 C CNN
+F 2 "" H 5850 2600 60  0001 C CNN
+F 3 "" H 5850 2600 60  0001 C CNN
+	1    5850 2600
 	0    -1   -1   0
 $EndComp
 $Comp
-L USB_2 J1
+L USB_A J1
 U 1 1 4E27DE01
-P 9850 5000
-F 0 "J1" H 9775 5250 60  0000 C CNN
-F 1 "USB_A" H 9900 4700 60  0001 C CNN
-F 2 "" H 9850 5000 60  0001 C CNN
-F 3 "" H 9850 5000 60  0001 C CNN
-F 4 "VCC" H 10175 5150 50  0001 C CNN "VCC"
-F 5 "D+" H 10150 5050 50  0001 C CNN "Data+"
-F 6 "D-" H 10150 4950 50  0001 C CNN "Data-"
-F 7 "GND" H 10175 4850 50  0001 C CNN "Ground"
-	1    9850 5000
-	-1   0    0    -1
+P 9950 5050
+F 0 "J1" H 9875 5300 60  0000 C CNN
+F 1 "USB_A" H 10000 4750 60  0001 C CNN
+F 2 "" H 9950 5050 60  0001 C CNN
+F 3 "" H 9950 5050 60  0001 C CNN
+F 4 "VCC" H 10275 5200 50  0001 C CNN "VCC"
+F 5 "D+" H 10250 5100 50  0001 C CNN "Data+"
+F 6 "D-" H 10250 5000 50  0001 C CNN "Data-"
+F 7 "GND" H 10275 4900 50  0001 C CNN "Ground"
+	1    9950 5050
+	0    1    1    0
 $EndComp
 Text Label 9500 5300 2    60   ~ 0
