File: fst-01.sch (KiCad schematic (older format))
At the start: 22 parts, among them J1 USB_A, K1 CONN_3, K2 CONN_2, K3 CONN_2, U1 STM32F103TB, U2 CAT6217-330, U3 NUF2221W1, U4 SST25VF032B, X1 12MHz

Commit message: fix connections of schematic
Connections:
- wire segments 108 -> 118
Changed lines of the file:
@@
 	2450 4300 2450 4450
 Wire Wire Line
-	3950 4950 3950 6100
-Wire Wire Line
-	3950 6100 3475 6100
+	3950 4950 3950 6150
+Wire Wire Line
+	3950 6150 3325 6150
 Wire Wire Line
 	4800 5800 4050 5800
 Wire Wire Line
-	2800 5625 2800 5525
+	2800 5525 2800 5675
 Connection ~ 6450 5450
 Wire Wire Line
@@
 	5600 5850 5600 5800
 Wire Wire Line
-	6450 5450 6450 5350
+	6450 5350 6450 5500
 Wire Wire Line
 	3950 4450 3200 4450
@@
 	7550 4850 7550 4550
 Wire Wire Line
-	5300 6300 5975 6300
+	5300 6300 6075 6300
 Wire Wire Line
 	5950 2800 5950 3400
 Wire Wire Line
-	7550 2250 7050 2250
+	7050 2250 7550 2250
 Wire Wire Line
 	7550 3650 7750 3650
@@
 	4900 3300 4900 3025
 Wire Wire Line
-	3200 5450 3200 5550
+	3200 5400 3200 5550
 Wire Wire Line
 	3950 4350 3100 4350
 Wire Wire Line
-	6450 4050 6450 4050
+	6450 4050 6500 4050
 Connection ~ 3500 4950
 Wire Wire Line
@@
 Connection ~ 6850 4050
 Wire Wire Line
-	7050 4050 6850 4050
+	6800 4050 7050 4050
 Wire Wire Line
 	7050 4050 7050 4150
@@
 Connection ~ 6450 4050
 Wire Wire Line
-	2450 4600 2375 4600
+	2375 4600 2500 4600
 Wire Wire Line
 	2375 4600 2375 4750
 Connection ~ 2850 4600
 Wire Wire Line
-	2850 4600 3100 4600
+	2800 4600 3100 4600
 Wire Wire Line
 	3100 4600 3100 4350
@@
 	3100 4000 3100 4250
 Wire Wire Line
-	3100 4000 2850 4000
+	2800 4000 3100 4000
 Connection ~ 2850 4000
 Wire Wire Line
 	2375 4150 2375 4000
 Wire Wire Line
-	2375 4000 2450 4000
+	2375 4000 2500 4000
 Connection ~ 7200 2250
 Wire Wire Line
 	8150 2250 8150 2400
 Wire Wire Line
-	7950 3750 7950 3800
-Wire Wire Line
-	7200 2700 7200 2650
+	7950 3700 7950 3800
+Wire Wire Line
+	7200 2700 7200 2600
 Wire Wire Line
 	3450 4050 3450 3950
 Wire Wire Line
-	3450 3950 3550 3950
+	3450 3950 3600 3950
 Wire Wire Line
 	3950 4650 3800 4650
@@
 	5050 3025 5050 3075
 Wire Wire Line
-	6475 6300 6550 6300
+	6375 6300 6550 6300
 Wire Wire Line
 	9500 5300 9500 5150
@@
 	7650 3350 7650 3500
 Wire Wire Line
-	3950 4150 3950 3900
-Wire Wire Line
-	7750 4300 7750 3350
+	3950 3900 3950 4150
+Wire Wire Line
+	7750 3350 7750 4300
 Connection ~ 7750 3650
 Wire Wire Line
@@
 	9200 4950 8950 4950
 Wire Wire Line
-	3200 4450 3200 5050
-Wire Wire Line
-	6450 5850 6450 5950
+	3200 4450 3200 5100
+Wire Wire Line
+	6450 5800 6450 5950
 Connection ~ 6450 5850
 Connection ~ 3950 3950
@@
 	5850 3300 5850 2800
 Wire Wire Line
-	2800 5825 2800 5950
-Wire Wire Line
-	3475 6300 4050 6300
-Wire Wire Line
-	4050 6300 4050 5800
+	2800 5775 2800 5950
+Wire Wire Line
+	3325 6250 4050 6250
+Wire Wire Line
+	4050 6250 4050 5800
 Wire Wire Line
 	5000 5800 5000 6950
@@
 	5100 6570 5100 5800
 Wire Wire Line
-	4290 6850 4290 6710
+	4290 6710 4290 6850
 Connection ~ 4290 6760
 Wire Wire Line
 	5300 5800 5300 6300
 Wire Wire Line
-	4150 7500 4150 7400
-Wire Wire Line
-	4150 7400 3950 7400
+	4150 7400 4150 7500
+Wire Wire Line
+	3900 7400 4150 7400
 $Comp
 L +3V3 #PWR01
@@
 	1    0    0    -1
 $EndComp
+Wire Wire Line
+	7200 2300 7200 2250
+Wire Wire Line
+	7750 2250 7800 2250
+Wire Wire Line
+	8100 2250 8150 2250
+Wire Wire Line
+	7950 3350 7950 3400
+Wire Wire Line
+	3950 3950 3900 3950
+Wire Wire Line
+	3500 4600 3500 4550
+Wire Wire Line
+	3500 4900 3500 4950
+Wire Wire Line
+	2800 5675 2650 5675
+Wire Wire Line
+	2650 5775 2800 5775
+Wire Wire Line
+	3600 7400 3550 7400
 $EndSCHEMATC
