File: fst-01.sch (KiCad schematic (older format))
At the start: 22 parts, among them J1 USB_A, K1 CONN_3, K2 CONN_2, K3 CONN_2, U1 STM32F103TB, U2 CAT6217-330, U3 NUF2221W1, U4 SST25VF032B, X1 12MHz

Commit message: fix direction of LED of schematic
Connections:
- wire segments 118 -> 132

Commit message: Fix schematic to FST-01G.
* Make Serial flash ROM optional.
* Connect USB connector's shield to GND.
* Remove USB_EN control.
Connections:
- net labels removed: USB_EN
- wire segments 132 -> 120
Other:
- note added: "Optional serial flash ROM"
Changed lines of the file:
@@
 	1    0    0    -1
 $EndComp
-Text Label 4580 6450 0    60   ~ 0
+Text Label 4350 6450 0    60   ~ 0
 NSS
 $Comp
@@
 	0    1    1    0
 $EndComp
-Text Label 4920 7040 0    60   ~ 0
+Text Label 4395 7040 0    60   ~ 0
 MOSI
-Text Label 4810 6950 0    60   ~ 0
+Text Label 4400 6950 0    60   ~ 0
 CLK
-Text Label 4640 6570 0    60   ~ 0
+Text Label 4450 6570 0    60   ~ 0
 MISO
 Text Label 4050 6050 1    60   ~ 0
@@
 Text Label 3950 5875 1    60   ~ 0
 PA2
-Text Label 7975 4650 0    60   ~ 0
-USB_EN
 $Comp
 L STM32F103TB U1
@@
 Connection ~ 3210 7040
 Wire Wire Line
-	3210 6950 3210 7040
-Wire Wire Line
-	3210 7040 3210 7140
+	3210 6950 3210 7140
 Wire Wire Line
 	4900 5800 4900 6450
@@
 	3550 3300 4800 3300
 Wire Wire Line
-	5600 5850 6100 5850
-Wire Wire Line
-	6100 5850 6450 5850
+	5600 5850 6450 5850
 Wire Wire Line
 	5600 5850 5600 5800
 Wire Wire Line
-	6450 5350 6450 5450
-Wire Wire Line
-	6450 5450 6450 5500
+	6450 5350 6450 5500
 Wire Wire Line
 	3950 4450 3200 4450
@@
 	5950 2800 5950 3400
 Wire Wire Line
-	7050 2250 7200 2250
-Wire Wire Line
-	7200 2250 7550 2250
+	7050 2250 7550 2250
 Wire Wire Line
 	7550 3650 7750 3650
@@
 	3300 4950 3300 4900
 Wire Wire Line
-	3300 4950 3500 4950
-Wire Wire Line
-	3500 4950 3800 4950
+	3300 4950 3800 4950
 Connection ~ 3700 4550
 Wire Wire Line
-	3500 4550 3700 4550
-Wire Wire Line
-	3700 4550 3950 4550
+	3500 4550 3950 4550
 Wire Wire Line
 	3700 4650 3700 4550
 Connection ~ 6850 4050
 Wire Wire Line
-	6800 4050 6850 4050
-Wire Wire Line
-	6850 4050 7050 4050
+	6800 4050 7050 4050
 Wire Wire Line
 	7050 4050 7050 4150
@@
 Connection ~ 2850 4600
 Wire Wire Line
-	2800 4600 2850 4600
-Wire Wire Line
-	2850 4600 3100 4600
+	2800 4600 3100 4600
 Wire Wire Line
 	3100 4600 3100 4350
@@
 	3100 4000 3100 4250
 Wire Wire Line
-	2800 4000 2850 4000
-Wire Wire Line
-	2850 4000 3100 4000
+	2800 4000 3100 4000
 Connection ~ 2850 4000
 Wire Wire Line
@@
 	3450 4050 3450 3950
 Wire Wire Line
-	3450 3950 3550 3950
-Wire Wire Line
-	3550 3950 3600 3950
+	3450 3950 3600 3950
 Wire Wire Line
 	3950 4650 3800 4650
@@
 	3100 4250 3950 4250
 Wire Wire Line
-	6450 3900 6450 4050
-Wire Wire Line
-	6450 4050 6450 4150
+	6450 3900 6450 4150
 Wire Wire Line
 	5500 5800 5500 5950
@@
 	7650 3350 7650 3500
 Wire Wire Line
-	3950 3900 3950 3950
-Wire Wire Line
-	3950 3950 3950 4150
-Wire Wire Line
-	7750 3350 7750 3650
-Wire Wire Line
-	7750 3650 7750 4300
+	3950 3900 3950 4150
+Wire Wire Line
+	7750 3350 7750 4300
 Connection ~ 7750 3650
 Wire Wire Line
@@
 	8950 5050 9650 5050
 Wire Wire Line
-	6450 4650 9200 4650
-Wire Wire Line
 	9200 4650 9200 4950
 Wire Wire Line
@@
 	3200 4450 3200 5100
 Wire Wire Line
-	6450 5800 6450 5850
-Wire Wire Line
-	6450 5850 6450 5950
+	6450 5800 6450 5950
 Connection ~ 6450 5850
 Connection ~ 3950 3950
@@
 	5100 6570 5100 5800
 Wire Wire Line
-	4290 6710 4290 6760
-Wire Wire Line
-	4290 6760 4290 6850
+	4290 6710 4290 6850
 Connection ~ 4290 6760
 Wire Wire Line
 	5300 5800 5300 6300
 Wire Wire Line
-	4150 7500 4150 7400
-Wire Wire Line
-	4150 7400 3950 7400
+	4150 7400 4150 7500
+Wire Wire Line
+	3900 7400 4150 7400
 Wire Wire Line
 	7200 2300 7200 2250
@@
 Wire Wire Line
 	2650 5775 2800 5775
+Wire Wire Line
+	3550 7400 3600 7400
+Wire Notes Line
+	2700 6375 4725 6375
+Wire Notes Line
+	4725 6375 4725 7700
+Wire Notes Line
+	4725 7700 2700 7700
+Wire Notes Line
+	2700 7700 2700 6375
+Text Notes 2750 7675 0    60   ~ 0
+Optional serial flash ROM
+$Comp
+L +3V3 #PWR?
+U 1 1 57C41036
+P 9200 4650
+F 0 "#PWR?" H 9200 4610 30  0001 C CNN
+F 1 "+3V3" H 9200 4760 30  0000 C CNN
+F 2 "" H 9200 4650 60  0001 C CNN
+F 3 "" H 9200 4650 60  0001 C CNN
+	1    9200 4650
+	1    0    0    -1
+$EndComp
+Wire Wire Line
+	10050 5350 9860 5350
+Wire Wire Line
+	9860 5350 9860 5305
+Wire Wire Line
+	9860 5305 9500 5305
+Connection ~ 9500 5300
 $EndSCHEMATC

Commit message: change LDO to LP2985-33
Parts:
- U2: value CAT6217-330 -> LP2985-33DBVR; symbol CAT6217-330 -> LP2985-33
Changed lines of the file:
@@
 LIBS:nuf2221w1
 LIBS:stm32f103
-LIBS:cat6217-330
-LIBS:stf202
 LIBS:power
 LIBS:device
 LIBS:conn
 LIBS:sst25vf032b
+LIBS:lp2985-33
 LIBS:fst-01-cache
 EELAYER 25 0
@@
 $EndComp
 $Comp
-L CAT6217-330 U2
+L LP2985-33 U2
 U 1 1 4E2CD88E
 P 7650 2800
 F 0 "U2" H 7400 3050 60  0000 C CNN
-F 1 "CAT6217-330" H 7650 2525 60  0000 C CNN
+F 1 "LP2985-33DBVR" H 7650 2525 60  0000 C CNN
 F 2 "" H 7650 2800 60  0001 C CNN
 F 3 "" H 7650 2800 60  0001 C CNN

Commit message: Update sch and net
Parts:
- C1, C11, C2, C3, C4, C5, C6, C7, C9: footprint (none) -> FST:c_0402
- C10, C8: footprint (none) -> FST:c_0603
- D1: footprint (none) -> FST:LED0603
- J1: footprint (none) -> FST:USB-A-PLUG
- K1: footprint (none) -> FST:SIL-3-2
- K2: footprint (none) -> FST:SIL-2-0
- K3: footprint (none) -> FST:SIL-2-2
- R1: footprint (none) -> FST:r_0402
- U1: footprint (none) -> FST:QFN36
- U2: footprint (none) -> FST:SOT23-5
- U3: footprint (none) -> FST:SOT363
- U4: footprint (none) -> FST:WSON8
- X1: footprint (none) -> FST:ABM8G
Changed lines of the file:
@@
 F 0 "K3" V 3075 6200 40  0000 C CNN
 F 1 "CONN_2" V 3175 6200 40  0000 C CNN
-F 2 "" H 3125 6200 60  0001 C CNN
+F 2 "FST:SIL-2-2" H 3125 6200 60  0001 C CNN
 F 3 "" H 3125 6200 60  0001 C CNN
 	1    3125 6200
@@
 F 0 "K2" V 2400 5725 40  0000 C CNN
 F 1 "CONN_2" V 2500 5725 40  0000 C CNN
-F 2 "" H 2450 5725 60  0001 C CNN
+F 2 "FST:SIL-2-0" H 2450 5725 60  0001 C CNN
 F 3 "" H 2450 5725 60  0001 C CNN
 	1    2450 5725
@@
 F 0 "C11" V 3650 7550 50  0000 L CNN
 F 1 "0.1uF" V 3800 7600 50  0000 L CNN
-F 2 "" H 3750 7400 60  0001 C CNN
+F 2 "FST:c_0402" H 3750 7400 60  0001 C CNN
 F 3 "" H 3750 7400 60  0001 C CNN
 	1    3750 7400
@@
 F 0 "U4" H 3750 6630 60  0000 C CNN
 F 1 "SST25VF032B" H 3750 7165 60  0000 C CNN
-F 2 "" H 3750 6900 60  0001 C CNN
+F 2 "FST:WSON8" H 3750 6900 60  0001 C CNN
 F 3 "" H 3750 6900 60  0001 C CNN
 	1    3750 6900
@@
 F 0 "X1" H 2850 4450 60  0000 C CNN
 F 1 "12MHz" H 2850 4150 60  0000 C CNN
-F 2 "" H 2850 4300 60  0001 C CNN
+F 2 "FST:ABM8G" H 2850 4300 60  0001 C CNN
 F 3 "" H 2850 4300 60  0001 C CNN
 	1    2850 4300
@@
 F 0 "U1" H 4300 5700 60  0000 C CNN
 F 1 "STM32F103TB" H 5150 4800 60  0000 C CNN
-F 2 "" H 5200 4550 60  0001 C CNN
+F 2 "FST:QFN36" H 5200 4550 60  0001 C CNN
 F 3 "" H 5200 4550 60  0001 C CNN
 	1    5200 4550
@@
 F 0 "U3" H 8250 5150 70  0000 C CNN
 F 1 "NUF2221W1" H 8450 4725 70  0000 C CNN
-F 2 "" H 8450 4950 60  0001 C CNN
+F 2 "FST:SOT363" H 8450 4950 60  0001 C CNN
 F 3 "" H 8450 4950 60  0001 C CNN
 	1    8450 4950
@@
 F 0 "K1" V 5800 2600 50  0000 C CNN
 F 1 "CONN_3" V 5900 2600 40  0000 C CNN
-F 2 "" H 5850 2600 60  0001 C CNN
+F 2 "FST:SIL-3-2" H 5850 2600 60  0001 C CNN
 F 3 "" H 5850 2600 60  0001 C CNN
 	1    5850 2600
@@
 F 0 "J1" H 9875 5300 60  0000 C CNN
 F 1 "USB_A" H 10000 4750 60  0001 C CNN
-F 2 "" H 9950 5050 60  0001 C CNN
+F 2 "FST:USB-A-PLUG" H 9950 5050 60  0001 C CNN
 F 3 "" H 9950 5050 60  0001 C CNN
 F 4 "VCC" H 10275 5200 50  0001 C CNN "VCC"
@@
 F 0 "C10" H 8000 3650 50  0000 L CNN
 F 1 "4.7uF" H 8000 3450 50  0000 L CNN
-F 2 "" H 7950 3550 60  0001 C CNN
+F 2 "FST:c_0603" H 7950 3550 60  0001 C CNN
 F 3 "" H 7950 3550 60  0001 C CNN
 	1    7950 3550
@@
 F 0 "C8" H 7250 2550 50  0000 L CNN
 F 1 "4.7uF" H 7250 2350 50  0000 L CNN
-F 2 "" H 7200 2450 60  0001 C CNN
+F 2 "FST:c_0603" H 7200 2450 60  0001 C CNN
 F 3 "" H 7200 2450 60  0001 C CNN
 	1    7200 2450
@@
 F 0 "D1" H 6550 6600 50  0000 C CNN
 F 1 "LED" H 6550 6400 50  0000 C CNN
-F 2 "" H 6550 6500 60  0001 C CNN
+F 2 "FST:LED0603" H 6550 6500 60  0001 C CNN
 F 3 "" H 6550 6500 60  0001 C CNN
 	1    6550 6500
@@
 F 0 "R1" V 6305 6300 50  0000 C CNN
 F 1 "510" V 6225 6300 50  0000 C CNN
-F 2 "" H 6225 6300 60  0001 C CNN
+F 2 "FST:r_0402" H 6225 6300 60  0001 C CNN
 F 3 "" H 6225 6300 60  0001 C CNN
 	1    6225 6300
@@
 F 0 "C3" H 3250 5350 50  0000 L CNN
 F 1 "0.1uF" H 3250 5150 50  0000 L CNN
-F 2 "" H 3200 5250 60  0001 C CNN
+F 2 "FST:c_0402" H 3200 5250 60  0001 C CNN
 F 3 "" H 3200 5250 60  0001 C CNN
 	1    3200 5250
@@
 F 0 "C6" H 6500 5750 50  0000 L CNN
 F 1 "0.1uF" H 6500 5550 50  0000 L CNN
-F 2 "" H 6450 5650 60  0001 C CNN
+F 2 "FST:c_0402" H 6450 5650 60  0001 C CNN
 F 3 "" H 6450 5650 60  0001 C CNN
 	1    6450 5650
@@
 F 0 "C4" H 3550 4850 50  0000 L CNN
 F 1 "0.1uF" H 3550 4650 50  0000 L CNN
-F 2 "" H 3500 4750 60  0001 C CNN
+F 2 "FST:c_0402" H 3500 4750 60  0001 C CNN
 F 3 "" H 3500 4750 60  0001 C CNN
 	1    3500 4750
@@
 F 0 "C5" H 3800 4050 50  0000 L CNN
 F 1 "0.1uF" H 3800 3850 50  0000 L CNN
-F 2 "" H 3750 3950 60  0001 C CNN
+F 2 "FST:c_0402" H 3750 3950 60  0001 C CNN
 F 3 "" H 3750 3950 60  0001 C CNN
 	1    3750 3950
@@
 F 0 "C7" H 6700 4150 50  0000 L CNN
 F 1 "0.1uF" H 6700 3950 50  0000 L CNN
-F 2 "" H 6650 4050 60  0001 C CNN
+F 2 "FST:c_0402" H 6650 4050 60  0001 C CNN
 F 3 "" H 6650 4050 60  0001 C CNN
 	1    6650 4050
@@
 F 0 "C9" H 8000 2350 50  0000 L CNN
 F 1 "0.01uF" H 8000 2150 50  0000 L CNN
-F 2 "" H 7950 2250 60  0001 C CNN
+F 2 "FST:c_0402" H 7950 2250 60  0001 C CNN
 F 3 "" H 7950 2250 60  0001 C CNN
 	1    7950 2250
@@
 F 0 "U2" H 7400 3050 60  0000 C CNN
 F 1 "LP2985-33DBVR" H 7650 2525 60  0000 C CNN
-F 2 "" H 7650 2800 60  0001 C CNN
+F 2 "FST:SOT23-5" H 7650 2800 60  0001 C CNN
 F 3 "" H 7650 2800 60  0001 C CNN
 	1    7650 2800
@@
 F 0 "C2" H 2700 4700 50  0000 L CNN
 F 1 "27pF" H 2700 4500 50  0000 L CNN
-F 2 "" H 2650 4600 60  0001 C CNN
+F 2 "FST:c_0402" H 2650 4600 60  0001 C CNN
 F 3 "" H 2650 4600 60  0001 C CNN
 	1    2650 4600
@@
 F 0 "C1" H 2700 4100 50  0000 L CNN
 F 1 "27pF" H 2700 3900 50  0000 L CNN
-F 2 "" H 2650 4000 60  0001 C CNN
+F 2 "FST:c_0402" H 2650 4000 60  0001 C CNN
 F 3 "" H 2650 4000 60  0001 C CNN
 	1    2650 4000
@@
 Optional serial flash ROM
 $Comp
-L +3V3 #PWR?
+L +3V3 #PWR030
 U 1 1 57C41036
 P 9200 4650
-F 0 "#PWR?" H 9200 4610 30  0001 C CNN
+F 0 "#PWR030" H 9200 4610 30  0001 C CNN
 F 1 "+3V3" H 9200 4760 30  0000 C CNN
 F 2 "" H 9200 4650 60  0001 C CNN
