File: fst-01.sch (KiCad schematic (older format))
At the start: 22 parts, among them J1 USB_A, K1 CONN_3, K2 CONN_2, K3 CONN_2, U1 STM32F103TB, U2 LP2985-33DBVR, U3 NUF2221W1, U4 SST25VF032B, X1 12MHz

Commit message: fst-01sz.
Parts:
- removed C11: 0.1uF, FST:c_0402, symbol C
- removed C9: 0.01uF, FST:c_0402, symbol C
- removed K2: CONN_2, FST:SIL-2-0, symbol CONN_01X02
- removed K3: CONN_2, FST:SIL-2-2, symbol CONN_01X02
- removed U4: SST25VF032B, FST:WSON8, symbol SST25VF032B
- C1, C2, C3, C4, C5, C6, C7: symbol C -> fst-01-rescue:C
- C8: symbol CP1 -> fst-01-rescue:CP1
- C9: renamed from C10; symbol CP1 -> fst-01-rescue:CP1
- D1: symbol LED -> fst-01-rescue:LED
- J1: symbol USB_A -> fst-01-rescue:USB_A
- K1: symbol CONN_01X03 -> Connector_Generic:Conn_01x05
- R1: symbol R -> fst-01-rescue:R
- U1: symbol STM32F103TB -> stm32f103:STM32F103TB
- U2: value LP2985-33DBVR -> MCP1700-3302E; footprint FST:SOT23-5 -> Package_TO_SOT_SMD:SOT-23; symbol LP2985-33 -> Regulator_Linear:MCP1700-3302E_SOT23
- U3: symbol NUF2221W1 -> nuf2221w1:NUF2221W1
- X1: symbol CRYSTAL -> crystal-gnd:CRYSTAL
Connections:
- net labels removed: CLK, MISO, MOSI, NSS, PA2
- wire segments 120 -> 112
Other:
- note removed: "Optional serial flash ROM"
- moved on the sheet: C9, D1, R1

Commit message: More change.
Parts:
- renumbered C4 to C1, C1 to C3, C5 to C4, C3 to C5, C7 to C6, C6 to C7
Changed lines of the file:
@@
 Sheet 1 1
 Title ""
-Date "2016-08-31"
-Rev "G"
-Comp ""
+Date "2018-08-08"
+Rev "SZ"
+Comp "Flying Stone Technology"
 Comment1 ""
 Comment2 ""
@@
 $EndComp
 $Comp
-L fst-01-rescue:C C3
+L fst-01-rescue:C C5
 U 1 1 4E2D6A2C
 P 3200 5250
-F 0 "C3" H 3250 5350 50  0000 L CNN
+F 0 "C5" H 3250 5350 50  0000 L CNN
 F 1 "0.1uF" H 3250 5150 50  0000 L CNN
 F 2 "FST:c_0402" H 3200 5250 60  0001 C CNN
@@
 $EndComp
 $Comp
-L fst-01-rescue:C C6
+L fst-01-rescue:C C7
 U 1 1 4E2D6573
 P 6450 5650
-F 0 "C6" H 6500 5750 50  0000 L CNN
+F 0 "C7" H 6500 5750 50  0000 L CNN
 F 1 "0.1uF" H 6500 5550 50  0000 L CNN
 F 2 "FST:c_0402" H 6450 5650 60  0001 C CNN
@@
 $EndComp
 $Comp
-L fst-01-rescue:C C4
+L fst-01-rescue:C C1
 U 1 1 4E2D63F9
 P 3500 4750
-F 0 "C4" H 3550 4850 50  0000 L CNN
+F 0 "C1" H 3550 4850 50  0000 L CNN
 F 1 "0.1uF" H 3550 4650 50  0000 L CNN
 F 2 "FST:c_0402" H 3500 4750 60  0001 C CNN
@@
 $EndComp
 $Comp
-L fst-01-rescue:C C5
+L fst-01-rescue:C C4
 U 1 1 4E2D167B
 P 3750 3950
-F 0 "C5" H 3800 4050 50  0000 L CNN
+F 0 "C4" H 3800 4050 50  0000 L CNN
 F 1 "0.1uF" H 3800 3850 50  0000 L CNN
 F 2 "FST:c_0402" H 3750 3950 60  0001 C CNN
@@
 $EndComp
 $Comp
-L fst-01-rescue:C C7
+L fst-01-rescue:C C6
 U 1 1 4E2D1296
 P 6650 4050
-F 0 "C7" H 6700 4150 50  0000 L CNN
+F 0 "C6" H 6700 4150 50  0000 L CNN
 F 1 "0.1uF" H 6700 3950 50  0000 L CNN
 F 2 "FST:c_0402" H 6650 4050 60  0001 C CNN
@@
 $EndComp
 $Comp
-L fst-01-rescue:C C1
+L fst-01-rescue:C C3
 U 1 1 4E2CD2B1
 P 2650 4000
-F 0 "C1" H 2700 4100 50  0000 L CNN
+F 0 "C3" H 2700 4100 50  0000 L CNN
 F 1 "27pF" H 2700 3900 50  0000 L CNN
 F 2 "FST:c_0402" H 2650 4000 60  0001 C CNN

Commit message: Add hole sensor, drv5032.
Parts:
- added U4: DRV5032FA, symbol drv5032:DRV5032
Connections:
- wire segments 112 -> 113
Changed lines of the file:
@@
 	5850 3300 5850 2300
 Wire Wire Line
-	3325 5925 4050 5925
-Wire Wire Line
-	4050 5925 4050 5800
+	4050 6300 4050 5800
 Wire Wire Line
 	7200 2300 7200 2250
@@
 Wire Wire Line
 	7250 4850 7250 6300
+$Comp
+L drv5032:DRV5032 U4
+U 1 1 5B6ADB25
+P 2975 6400
+F 0 "U4" H 2745 6446 50  0000 R CNN
+F 1 "DRV5032FA" H 2745 6355 50  0000 R CNN
+F 2 "" H 2975 6050 50  0001 L CIN
+F 3 " " H 2875 6400 50  0001 C CNN
+	1    2975 6400
+	1    0    0    -1
+$EndComp
+Wire Wire Line
+	3275 6300 4050 6300
+$Comp
+L power:GND #PWR?
+U 1 1 5B6C3332
+P 2875 6800
+F 0 "#PWR?" H 2875 6800 30  0001 C CNN
+F 1 "GND" H 2875 6730 30  0001 C CNN
+F 2 "" H 2875 6800 60  0001 C CNN
+F 3 "" H 2875 6800 60  0001 C CNN
+	1    2875 6800
+	1    0    0    -1
+$EndComp
+$Comp
+L power:+3V3 #PWR?
+U 1 1 5B6C34FF
+P 2875 5900
+F 0 "#PWR?" H 2875 5860 30  0001 C CNN
+F 1 "+3V3" H 2875 6010 30  0000 C CNN
+F 2 "" H 2875 5900 60  0001 C CNN
+F 3 "" H 2875 5900 60  0001 C CNN
+	1    2875 5900
+	1    0    0    -1
+$EndComp
+Wire Wire Line
+	2875 6000 2875 5900
 $EndSCHEMATC

Commit message: More change to PCBA.
Parts:
- U4: footprint (none) -> X2SON
Changed lines of the file:
@@
 F 0 "U4" H 2745 6446 50  0000 R CNN
 F 1 "DRV5032FA" H 2745 6355 50  0000 R CNN
-F 2 "" H 2975 6050 50  0001 L CIN
+F 2 "X2SON" H 2975 6050 50  0001 L CIN
 F 3 " " H 2875 6400 50  0001 C CNN
 	1    2975 6400

Commit message: change parts.
Parts:
- removed C2, C3: 27pF, FST:c_0402, symbol fst-01-rescue:C
- R1: value 510 -> 470
- renumbered C4 to C2, C5 to C3, C6 to C4, C7 to C5, C8 to C6, C9 to C7
Connections:
- wire segments 113 -> 107
Changed lines of the file:
@@
 Sheet 1 1
 Title ""
-Date "2018-08-08"
+Date "2018-08-15"
 Rev "SZ"
 Comp "Flying Stone Technology"
@@
 L power:GND #PWR05
 U 1 1 4E82CDD0
-P 2450 4450
-F 0 "#PWR05" H 2450 4450 30  0001 C CNN
-F 1 "GND" H 2450 4380 30  0001 C CNN
-F 2 "" H 2450 4450 60  0001 C CNN
-F 3 "" H 2450 4450 60  0001 C CNN
-	1    2450 4450
+P 2400 4450
+F 0 "#PWR05" H 2400 4450 30  0001 C CNN
+F 1 "GND" H 2400 4380 30  0001 C CNN
+F 2 "" H 2400 4450 60  0001 C CNN
+F 3 "" H 2400 4450 60  0001 C CNN
+	1    2400 4450
 	1    0    0    -1
 $EndComp
@@
 L crystal-gnd:CRYSTAL X1
 U 1 1 4E82CD9F
-P 2850 4300
-F 0 "X1" H 2850 4450 60  0000 C CNN
-F 1 "12MHz" H 2850 4150 60  0000 C CNN
-F 2 "FST:ABM8G" H 2850 4300 60  0001 C CNN
-F 3 "" H 2850 4300 60  0001 C CNN
-	1    2850 4300
+P 2800 4300
+F 0 "X1" H 2800 4450 60  0000 C CNN
+F 1 "12MHz" H 2800 4150 60  0000 C CNN
+F 2 "FST:ABM8G" H 2800 4300 60  0001 C CNN
+F 3 "" H 2800 4300 60  0001 C CNN
+	1    2800 4300
 	0    1    1    0
 $EndComp
@@
 SWCLK
 $Comp
-L fst-01-rescue:CP1 C9
+L fst-01-rescue:CP1 C7
 U 1 1 4E2D79C8
 P 8350 2450
-F 0 "C9" H 8400 2550 50  0000 L CNN
+F 0 "C7" H 8400 2550 50  0000 L CNN
 F 1 "4.7uF" H 8400 2350 50  0000 L CNN
 F 2 "FST:c_0603" H 8350 2450 60  0001 C CNN
@@
 $EndComp
 $Comp
-L fst-01-rescue:CP1 C8
+L fst-01-rescue:CP1 C6
 U 1 1 4E2D79BC
 P 7200 2450
-F 0 "C8" H 7250 2550 50  0000 L CNN
+F 0 "C6" H 7250 2550 50  0000 L CNN
 F 1 "4.7uF" H 7250 2350 50  0000 L CNN
 F 2 "FST:c_0603" H 7200 2450 60  0001 C CNN
@@
 P 6550 6550
 F 0 "R1" V 6630 6550 50  0000 C CNN
-F 1 "510" V 6550 6550 50  0000 C CNN
+F 1 "470" V 6550 6550 50  0000 C CNN
 F 2 "FST:r_0402" H 6550 6550 60  0001 C CNN
 F 3 "" H 6550 6550 60  0001 C CNN
@@
 $EndComp
 $Comp
-L fst-01-rescue:C C5
+L fst-01-rescue:C C3
 U 1 1 4E2D6A2C
 P 3200 5250
-F 0 "C5" H 3250 5350 50  0000 L CNN
+F 0 "C3" H 3250 5350 50  0000 L CNN
 F 1 "0.1uF" H 3250 5150 50  0000 L CNN
 F 2 "FST:c_0402" H 3200 5250 60  0001 C CNN
@@
 $EndComp
 $Comp
-L fst-01-rescue:C C7
+L fst-01-rescue:C C5
 U 1 1 4E2D6573
 P 6450 5650
-F 0 "C7" H 6500 5750 50  0000 L CNN
+F 0 "C5" H 6500 5750 50  0000 L CNN
 F 1 "0.1uF" H 6500 5550 50  0000 L CNN
 F 2 "FST:c_0402" H 6450 5650 60  0001 C CNN
@@
 $EndComp
 $Comp
-L fst-01-rescue:C C4
+L fst-01-rescue:C C2
 U 1 1 4E2D167B
 P 3750 3950
-F 0 "C4" H 3800 4050 50  0000 L CNN
+F 0 "C2" H 3800 4050 50  0000 L CNN
 F 1 "0.1uF" H 3800 3850 50  0000 L CNN
 F 2 "FST:c_0402" H 3750 3950 60  0001 C CNN
@@
 $EndComp
 $Comp
-L fst-01-rescue:C C6
+L fst-01-rescue:C C4
 U 1 1 4E2D1296
 P 6650 4050
-F 0 "C6" H 6700 4150 50  0000 L CNN
+F 0 "C4" H 6700 4150 50  0000 L CNN
 F 1 "0.1uF" H 6700 3950 50  0000 L CNN
 F 2 "FST:c_0402" H 6650 4050 60  0001 C CNN
@@
 	-1   0    0    -1
 $EndComp
-$Comp
-L power:GND #PWR026
-U 1 1 4E2CD35B
-P 2375 4750
-F 0 "#PWR026" H 2375 4750 30  0001 C CNN
-F 1 "GND" H 2375 4680 30  0001 C CNN
-F 2 "" H 2375 4750 60  0001 C CNN
-F 3 "" H 2375 4750 60  0001 C CNN
-	1    2375 4750
-	1    0    0    -1
-$EndComp
-$Comp
-L power:GND #PWR027
-U 1 1 4E2CD351
-P 2375 4150
-F 0 "#PWR027" H 2375 4150 30  0001 C CNN
-F 1 "GND" H 2375 4080 30  0001 C CNN
-F 2 "" H 2375 4150 60  0001 C CNN
-F 3 "" H 2375 4150 60  0001 C CNN
-	1    2375 4150
-	1    0    0    -1
-$EndComp
-$Comp
-L fst-01-rescue:C C2
-U 1 1 4E2CD2C4
-P 2650 4600
-F 0 "C2" H 2700 4700 50  0000 L CNN
-F 1 "27pF" H 2700 4500 50  0000 L CNN
-F 2 "FST:c_0402" H 2650 4600 60  0001 C CNN
-F 3 "" H 2650 4600 60  0001 C CNN
-	1    2650 4600
-	0    1    1    0
-$EndComp
-$Comp
-L fst-01-rescue:C C3
-U 1 1 4E2CD2B1
-P 2650 4000
-F 0 "C3" H 2700 4100 50  0000 L CNN
-F 1 "27pF" H 2700 3900 50  0000 L CNN
-F 2 "FST:c_0402" H 2650 4000 60  0001 C CNN
-F 3 "" H 2650 4000 60  0001 C CNN
-	1    2650 4000
-	0    1    1    0
-$EndComp
 Text Label 9200 5050 0    60   ~ 0
 D+_PLUG
@@
 $EndComp
 Wire Wire Line
-	2450 4300 2450 4450
+	2400 4300 2400 4450
 Wire Wire Line
 	4800 5800 4050 5800
@@
 Connection ~ 6450 4050
 Wire Wire Line
-	2375 4600 2500 4600
-Wire Wire Line
-	2375 4600 2375 4750
-Connection ~ 2850 4600
-Wire Wire Line
-	2800 4600 2850 4600
-Wire Wire Line
 	3100 4600 3100 4350
 Wire Wire Line
@@
 Wire Wire Line
 	3100 4000 3100 4250
-Wire Wire Line
-	2800 4000 2850 4000
-Connection ~ 2850 4000
-Wire Wire Line
-	2375 4150 2375 4000
-Wire Wire Line
-	2375 4000 2500 4000
 Connection ~ 7200 2250
 Wire Wire Line
@@
 	6450 4050 6450 4150
 Wire Wire Line
-	2850 4600 3100 4600
-Wire Wire Line
-	2850 4000 3100 4000
-Wire Wire Line
 	7200 2250 7550 2250
 Wire Wire Line
@@
 Wire Wire Line
 	2875 6000 2875 5900
+Wire Wire Line
+	2800 4600 3100 4600
+Wire Wire Line
+	2800 4000 3100 4000
 $EndSCHEMATC

Commit message: Add position file and name change for U1 to GD.
Parts:
- U1: value STM32F103TB -> GD32F103TB
- X1: footprint FST:ABM8G -> FST:FA-20H
Changed lines of the file:
@@
 F 0 "X1" H 2800 4450 60  0000 C CNN
 F 1 "12MHz" H 2800 4150 60  0000 C CNN
-F 2 "FST:ABM8G" H 2800 4300 60  0001 C CNN
+F 2 "FST:FA-20H" H 2800 4300 60  0001 C CNN
 F 3 "" H 2800 4300 60  0001 C CNN
 	1    2800 4300
@@
 P 5200 4550
 F 0 "U1" H 4300 5700 60  0000 C CNN
-F 1 "STM32F103TB" H 5150 4800 60  0000 C CNN
+F 1 "GD32F103TB" H 5150 4800 60  0000 C CNN
 F 2 "FST:QFN36" H 5200 4550 60  0001 C CNN
 F 3 "" H 5200 4550 60  0001 C CNN
@@
 	3275 6300 4050 6300
 $Comp
-L power:GND #PWR?
+L power:GND #PWR0102
 U 1 1 5B6C3332
 P 2875 6800
-F 0 "#PWR?" H 2875 6800 30  0001 C CNN
+F 0 "#PWR0102" H 2875 6800 30  0001 C CNN
 F 1 "GND" H 2875 6730 30  0001 C CNN
 F 2 "" H 2875 6800 60  0001 C CNN
@@
 $EndComp
 $Comp
-L power:+3V3 #PWR?
+L power:+3V3 #PWR0103
 U 1 1 5B6C34FF
 P 2875 5900
-F 0 "#PWR?" H 2875 5860 30  0001 C CNN
+F 0 "#PWR0103" H 2875 5860 30  0001 C CNN
 F 1 "+3V3" H 2875 6010 30  0000 C CNN
 F 2 "" H 2875 5900 60  0001 C CNN

Commit message: Update PCBA.
Parts:
- J1: footprint FST:USB-A-PLUG -> FST:USB-A-ZT01
- K1: value CONN_3 -> CONN_5; footprint FST:SIL-3-2 -> FST:SIL-5
- U2: footprint Package_TO_SOT_SMD:SOT-23 -> FST-01:SOT-23
- U4: footprint X2SON -> FST-01:X2SON
Changed lines of the file:
@@
 P 5850 2100
 F 0 "K1" V 5800 2100 50  0000 C CNN
-F 1 "CONN_3" V 5900 2100 40  0000 C CNN
-F 2 "FST:SIL-3-2" H 5850 2100 60  0001 C CNN
+F 1 "CONN_5" V 5900 2100 40  0000 C CNN
+F 2 "FST:SIL-5" H 5850 2100 60  0001 C CNN
 F 3 "" H 5850 2100 60  0001 C CNN
 	1    5850 2100
@@
 F 0 "J1" H 9875 5300 60  0000 C CNN
 F 1 "USB_A" H 10000 4750 60  0001 C CNN
-F 2 "FST:USB-A-PLUG" H 9950 5050 60  0001 C CNN
+F 2 "FST:USB-A-ZT01" H 9950 5050 60  0001 C CNN
 F 3 "" H 9950 5050 60  0001 C CNN
 F 4 "VCC" H 10275 5200 50  0001 C CNN "VCC"
@@
 F 0 "U2" H 7600 2000 60  0000 C CNN
 F 1 "MCP1700-3302E" H 7850 2400 60  0000 C CNN
-F 2 "Package_TO_SOT_SMD:SOT-23" H 7850 2250 60  0001 C CNN
+F 2 "FST-01:SOT-23" H 7850 2250 60  0001 C CNN
 F 3 "http://ww1.microchip.com/downloads/en/DeviceDoc/20001826D.pdfhttp://ww1.microchip.com/downloads/en/DeviceDoc/20001826D.pdf" H 7850 2250 60  0001 C CNN
 	1    7850 2250
@@
 F 0 "U4" H 2745 6446 50  0000 R CNN
 F 1 "DRV5032FA" H 2745 6355 50  0000 R CNN
-F 2 "X2SON" H 2975 6050 50  0001 L CIN
+F 2 "FST-01:X2SON" H 2975 6050 50  0001 L CIN
 F 3 " " H 2875 6400 50  0001 C CNN
 	1    2975 6400
